File: Output Register.sch (KiCad schematic (older format))
At the start: 0 parts

Commit message: Add output display.
Parts:
- added C? (x2): 10nF, symbol Device:C_Small
- added R? (x2): 1kΩ, symbol Device:R_Small_US
- added U?: CC56-12CGKWA, Display_7Segment:CA56-12CGKWA, symbol Display_Character:CC56-12CGKWA
- added U?: 74LS139, symbol 74xx:74LS139
- added U?: 74LS393, symbol 74xx:74LS393
- added U?: LM555, symbol Timer:LM555
- added U?: 28C256, symbol Memory_EEPROM:28C256
Connections:
- new net: U?.1 (e), U?.13 (D2)
- new net: U?.10 (f), U?.12 (D1)
- new net: U?.11 (a), U?.18 (D6)
- new net: U?.12 (CC1), U?.7 (O3)
- new net: U?.15 (D3), U?.2 (d)
- new net: U?.19 (D7), U?.3 (DPX)
- new net: U?.16 (D4), U?.4 (c)
- new net: U?.11 (D0), U?.5 (g)
- new net: U?.4 (O0), U?.6 (CC4)
- new net: U?.17 (D5), U?.7 (b)
- new net: U?.5 (O1), U?.8 (CC3)
- new net: U?.6 (O2), U?.9 (CC2)
- new net: U?.2 (A0), U?.3 (Q0)
- new net: U?.3 (A1), U?.4 (Q1)
- new net: U?.1 (CP), U?.3 (Q)
- new net: C?.1, R?.2, U?.2 (TR), U?.6 (THR)
- new net: C?.2, U?.5 (CV)
- new net: R?.1, R?.2, U?.7 (DIS)
- new net GND: C?.1, C?.2, U?.1 (A14), U?.1 (E), U?.1 (GND), U?.14 (GND), U?.2 (A12), U?.2 (MR), U?.20 (~CS), U?.21 (A10), U?.22 (~OE), U?.23 (A11), U?.24 (A9), U?.25 (A8), U?.26 (A13)
- new net Out0: U?.10 (A0)
- new net Out1: U?.9 (A1)
- new net Out2: U?.8 (A2)
- new net Out3: U?.7 (A3)
- new net Out4: U?.6 (A4)
- new net Out5: U?.5 (A5)
- new net Out6: U?.4 (A6)
- new net Out7: U?.3 (A7)
- new net VCC: R?.1, U?.27 (~WE), U?.28 (VCC), U?.4 (R), U?.5 (Q2), U?.6 (Q3), U?.8 (VCC)
