File: Instruction ROM.sch (KiCad schematic (older format))
At the start: 0 parts

Commit message: Added schematic for Instruction ROM.
Parts:
- added U? (x2): GLS29EE010, symbol Memory_EEPROM:GLS29EE010
Connections:
- new net GND: U?.16 (VSS), U?.16 (VSS), U?.2 (A16), U?.2 (A16), U?.22 (CE), U?.22 (CE), U?.24 (OE), U?.24 (OE)
- new net IROM00: U?.13 (DQ0)
- new net IROM01: U?.14 (DQ1)
- new net IROM02: U?.15 (DQ2)
- new net IROM03: U?.17 (DQ3)
- new net IROM04: U?.18 (DQ4)
- new net IROM05: U?.19 (DQ5)
- new net IROM06: U?.20 (DQ6)
- new net IROM07: U?.21 (DQ7)
- new net IROM08: U?.13 (DQ0)
- new net IROM09: U?.14 (DQ1)
- new net IROM10: U?.15 (DQ2)
- new net IROM11: U?.17 (DQ3)
- new net IROM12: U?.18 (DQ4)
- new net IROM13: U?.19 (DQ5)
- new net IROM14: U?.20 (DQ6)
- new net IROM15: U?.21 (DQ7)
- new net PC00: U?.12 (A0), U?.12 (A0)
- new net PC01: U?.11 (A1), U?.11 (A1)
- new net PC02: U?.10 (A2), U?.10 (A2)
- new net PC03: U?.9 (A3), U?.9 (A3)
- new net PC04: U?.8 (A4), U?.8 (A4)
- new net PC05: U?.7 (A5), U?.7 (A5)
- new net PC06: U?.6 (A6), U?.6 (A6)
- new net PC07: U?.5 (A7), U?.5 (A7)
- new net PC08: U?.27 (A8), U?.27 (A8)
- new net PC09: U?.26 (A9), U?.26 (A9)
- new net PC10: U?.23 (A10), U?.23 (A10)
- new net PC11: U?.25 (A11), U?.25 (A11)
- new net PC12: U?.4 (A12), U?.4 (A12)
- new net PC13: U?.28 (A13), U?.28 (A13)
- new net PC14: U?.29 (A14), U?.29 (A14)
- new net PC15: U?.3 (A15), U?.3 (A15)
- new net VCC: U?.31 (WE), U?.31 (WE), U?.32 (VDD), U?.32 (VDD)
