File: Schematics/Control Word DIsplay.sch (KiCad schematic (older format))
At the start: 0 parts

Commit message: Flesh out the control signals in the execute unit.
Parts:
- added D? (x16): LED, symbol Device:LED
- added R? (x16): 220Ω, symbol Device:R
Connections:
- new net: D?.1 (K), R?.1 (x16)
- new net ControlWord00: D?.2 (A)
- new net ControlWord01: D?.2 (A)
- new net ControlWord02: D?.2 (A)
- new net ControlWord03: D?.2 (A)
- new net ControlWord04: D?.2 (A)
- new net ControlWord05: D?.2 (A)
- new net ControlWord06: D?.2 (A)
- new net ControlWord07: D?.2 (A)
- new net ControlWord08: D?.2 (A)
- new net ControlWord09: D?.2 (A)
- new net ControlWord10: D?.2 (A)
- new net ControlWord11: D?.2 (A)
- new net ControlWord12: D?.2 (A)
- new net ControlWord13: D?.2 (A)
- new net ControlWord14: D?.2 (A)
- new net ControlWord15: D?.2 (A)
- new net GND: R?.2, R?.2, R?.2, R?.2, R?.2, R?.2, R?.2, R?.2, R?.2, R?.2, R?.2, R?.2, R?.2, R?.2, R?.2, R?.2
Other:
- note added: "Control Word LED Indicators"
- note added: "TODO: These signals are active-low. The LEDs should be wired to light up when they go active."
