File: Schematics/Instruction Register.sch (KiCad schematic (older format))
At the start: 44 parts

Commit message: annotate
Parts:
- gave numbers to parts that had none: 44

Commit message: Add footprints to all decoupling caps
Parts:
- C39, C40, C41, C42, C43, C44: footprint (none) -> Capacitor_THT:C_Disc_D4.3mm_W1.9mm_P5.00mm
Changed lines of the file:
@@
 F 0 "C43" H 3965 7796 50  0000 L CNN
 F 1 "100nF" H 3965 7705 50  0000 L CNN
-F 2 "" H 3888 7600 50  0001 C CNN
+F 2 "Capacitor_THT:C_Disc_D4.3mm_W1.9mm_P5.00mm" H 3888 7600 50  0001 C CNN
 F 3 "~" H 3850 7750 50  0001 C CNN
 	1    3850 7750
@@
 F 0 "C42" H 3465 7796 50  0000 L CNN
 F 1 "100nF" H 3465 7705 50  0000 L CNN
-F 2 "" H 3388 7600 50  0001 C CNN
+F 2 "Capacitor_THT:C_Disc_D4.3mm_W1.9mm_P5.00mm" H 3388 7600 50  0001 C CNN
 F 3 "~" H 3350 7750 50  0001 C CNN
 	1    3350 7750
@@
 F 0 "C41" H 2965 7796 50  0000 L CNN
 F 1 "100nF" H 2965 7705 50  0000 L CNN
-F 2 "" H 2888 7600 50  0001 C CNN
+F 2 "Capacitor_THT:C_Disc_D4.3mm_W1.9mm_P5.00mm" H 2888 7600 50  0001 C CNN
 F 3 "~" H 2850 7750 50  0001 C CNN
 	1    2850 7750
@@
 F 0 "C40" H 2465 7796 50  0000 L CNN
 F 1 "100nF" H 2465 7705 50  0000 L CNN
-F 2 "" H 2388 7600 50  0001 C CNN
+F 2 "Capacitor_THT:C_Disc_D4.3mm_W1.9mm_P5.00mm" H 2388 7600 50  0001 C CNN
 F 3 "~" H 2350 7750 50  0001 C CNN
 	1    2350 7750
@@
 F 0 "C39" H 1965 7796 50  0000 L CNN
 F 1 "100nF" H 1965 7705 50  0000 L CNN
-F 2 "" H 1888 7600 50  0001 C CNN
+F 2 "Capacitor_THT:C_Disc_D4.3mm_W1.9mm_P5.00mm" H 1888 7600 50  0001 C CNN
 F 3 "~" H 1850 7750 50  0001 C CNN
 	1    1850 7750
@@
 F 0 "C44" H 4465 7796 50  0000 L CNN
 F 1 "100nF" H 4465 7705 50  0000 L CNN
-F 2 "" H 4388 7600 50  0001 C CNN
+F 2 "Capacitor_THT:C_Disc_D4.3mm_W1.9mm_P5.00mm" H 4388 7600 50  0001 C CNN
 F 3 "~" H 4350 7750 50  0001 C CNN
 	1    4350 7750

Commit message: Assign a bunch of part footprints.
Parts:
- D25, D26, D27, D28, D29, D30, D31, D32, D33, D34, D35, D36, D37, D38, D39, D40: footprint (none) -> LED_THT:LED_D5.0mm
- R25, R26, R27, R28, R29, R30, R31, R32, R33, R34, R35, R36, R37, R38, R39, R40: footprint (none) -> Resistor_THT:R_Axial_DIN0207_L6.3mm_D2.5mm_P7.62mm_Horizontal
Changed lines of the file:
@@
 F 0 "D29" V 2139 6483 50  0000 R CNN
 F 1 "LED" V 2048 6483 50  0000 R CNN
-F 2 "" H 2100 6600 50  0001 C CNN
+F 2 "LED_THT:LED_D5.0mm" H 2100 6600 50  0001 C CNN
 F 3 "~" H 2100 6600 50  0001 C CNN
 	1    2100 6600
@@
 F 0 "D30" V 2489 6483 50  0000 R CNN
 F 1 "LED" V 2398 6483 50  0000 R CNN
-F 2 "" H 2450 6600 50  0001 C CNN
+F 2 "LED_THT:LED_D5.0mm" H 2450 6600 50  0001 C CNN
 F 3 "~" H 2450 6600 50  0001 C CNN
 	1    2450 6600
@@
 F 0 "D31" V 2839 6483 50  0000 R CNN
 F 1 "LED" V 2748 6483 50  0000 R CNN
-F 2 "" H 2800 6600 50  0001 C CNN
+F 2 "LED_THT:LED_D5.0mm" H 2800 6600 50  0001 C CNN
 F 3 "~" H 2800 6600 50  0001 C CNN
 	1    2800 6600
@@
 F 0 "D32" V 3189 6483 50  0000 R CNN
 F 1 "LED" V 3098 6483 50  0000 R CNN
-F 2 "" H 3150 6600 50  0001 C CNN
+F 2 "LED_THT:LED_D5.0mm" H 3150 6600 50  0001 C CNN
 F 3 "~" H 3150 6600 50  0001 C CNN
 	1    3150 6600
@@
 F 0 "D28" V 1789 6483 50  0000 R CNN
 F 1 "LED" V 1698 6483 50  0000 R CNN
-F 2 "" H 1750 6600 50  0001 C CNN
+F 2 "LED_THT:LED_D5.0mm" H 1750 6600 50  0001 C CNN
 F 3 "~" H 1750 6600 50  0001 C CNN
 	1    1750 6600
@@
 F 0 "D27" V 1439 6483 50  0000 R CNN
 F 1 "LED" V 1348 6483 50  0000 R CNN
-F 2 "" H 1400 6600 50  0001 C CNN
+F 2 "LED_THT:LED_D5.0mm" H 1400 6600 50  0001 C CNN
 F 3 "~" H 1400 6600 50  0001 C CNN
 	1    1400 6600
@@
 F 0 "D26" V 1089 6483 50  0000 R CNN
 F 1 "LED" V 998 6483 50  0000 R CNN
-F 2 "" H 1050 6600 50  0001 C CNN
+F 2 "LED_THT:LED_D5.0mm" H 1050 6600 50  0001 C CNN
 F 3 "~" H 1050 6600 50  0001 C CNN
 	1    1050 6600
@@
 F 0 "D33" V 3539 6483 50  0000 R CNN
 F 1 "LED" V 3448 6483 50  0000 R CNN
-F 2 "" H 3500 6600 50  0001 C CNN
+F 2 "LED_THT:LED_D5.0mm" H 3500 6600 50  0001 C CNN
 F 3 "~" H 3500 6600 50  0001 C CNN
 	1    3500 6600
@@
 F 0 "D34" V 3889 6483 50  0000 R CNN
 F 1 "LED" V 3798 6483 50  0000 R CNN
-F 2 "" H 3850 6600 50  0001 C CNN
+F 2 "LED_THT:LED_D5.0mm" H 3850 6600 50  0001 C CNN
 F 3 "~" H 3850 6600 50  0001 C CNN
 	1    3850 6600
@@
 F 0 "D35" V 4239 6483 50  0000 R CNN
 F 1 "LED" V 4148 6483 50  0000 R CNN
-F 2 "" H 4200 6600 50  0001 C CNN
+F 2 "LED_THT:LED_D5.0mm" H 4200 6600 50  0001 C CNN
 F 3 "~" H 4200 6600 50  0001 C CNN
 	1    4200 6600
@@
 F 0 "D36" V 4589 6483 50  0000 R CNN
 F 1 "LED" V 4498 6483 50  0000 R CNN
-F 2 "" H 4550 6600 50  0001 C CNN
+F 2 "LED_THT:LED_D5.0mm" H 4550 6600 50  0001 C CNN
 F 3 "~" H 4550 6600 50  0001 C CNN
 	1    4550 6600
@@
 F 0 "D37" V 4939 6483 50  0000 R CNN
 F 1 "LED" V 4848 6483 50  0000 R CNN
-F 2 "" H 4900 6600 50  0001 C CNN
+F 2 "LED_THT:LED_D5.0mm" H 4900 6600 50  0001 C CNN
 F 3 "~" H 4900 6600 50  0001 C CNN
 	1    4900 6600
@@
 F 0 "D38" V 5289 6483 50  0000 R CNN
 F 1 "LED" V 5198 6483 50  0000 R CNN
-F 2 "" H 5250 6600 50  0001 C CNN
+F 2 "LED_THT:LED_D5.0mm" H 5250 6600 50  0001 C CNN
 F 3 "~" H 5250 6600 50  0001 C CNN
 	1    5250 6600
@@
 F 0 "D39" V 5639 6483 50  0000 R CNN
 F 1 "LED" V 5548 6483 50  0000 R CNN
-F 2 "" H 5600 6600 50  0001 C CNN
+F 2 "LED_THT:LED_D5.0mm" H 5600 6600 50  0001 C CNN
 F 3 "~" H 5600 6600 50  0001 C CNN
 	1    5600 6600
@@
 F 0 "D40" V 5989 6483 50  0000 R CNN
 F 1 "LED" V 5898 6483 50  0000 R CNN
-F 2 "" H 5950 6600 50  0001 C CNN
+F 2 "LED_THT:LED_D5.0mm" H 5950 6600 50  0001 C CNN
 F 3 "~" H 5950 6600 50  0001 C CNN
 	1    5950 6600
@@
 F 0 "R25" H 768 7096 50  0000 L CNN
 F 1 "220Ω" H 768 7005 50  0000 L CNN
-F 2 "" V 740 7040 50  0001 C CNN
+F 2 "Resistor_THT:R_Axial_DIN0207_L6.3mm_D2.5mm_P7.62mm_Horizontal" V 740 7040 50  0001 C CNN
 F 3 "~" H 700 7050 50  0001 C CNN
 	1    700  7050
@@
 F 0 "R26" H 1118 7096 50  0000 L CNN
 F 1 "220Ω" H 1118 7005 50  0000 L CNN
-F 2 "" V 1090 7040 50  0001 C CNN
+F 2 "Resistor_THT:R_Axial_DIN0207_L6.3mm_D2.5mm_P7.62mm_Horizontal" V 1090 7040 50  0001 C CNN
 F 3 "~" H 1050 7050 50  0001 C CNN
 	1    1050 7050
@@
 F 0 "R27" H 1468 7096 50  0000 L CNN
 F 1 "220Ω" H 1468 7005 50  0000 L CNN
-F 2 "" V 1440 7040 50  0001 C CNN
+F 2 "Resistor_THT:R_Axial_DIN0207_L6.3mm_D2.5mm_P7.62mm_Horizontal" V 1440 7040 50  0001 C CNN
 F 3 "~" H 1400 7050 50  0001 C CNN
 	1    1400 7050
@@
 F 0 "R28" H 1818 7096 50  0000 L CNN
 F 1 "220Ω" H 1818 7005 50  0000 L CNN
-F 2 "" V 1790 7040 50  0001 C CNN
+F 2 "Resistor_THT:R_Axial_DIN0207_L6.3mm_D2.5mm_P7.62mm_Horizontal" V 1790 7040 50  0001 C CNN
 F 3 "~" H 1750 7050 50  0001 C CNN
 	1    1750 7050
@@
 F 0 "R29" H 2168 7096 50  0000 L CNN
 F 1 "220Ω" H 2168 7005 50  0000 L CNN
-F 2 "" V 2140 7040 50  0001 C CNN
+F 2 "Resistor_THT:R_Axial_DIN0207_L6.3mm_D2.5mm_P7.62mm_Horizontal" V 2140 7040 50  0001 C CNN
 F 3 "~" H 2100 7050 50  0001 C CNN
 	1    2100 7050
@@
 F 0 "R30" H 2518 7096 50  0000 L CNN
 F 1 "220Ω" H 2518 7005 50  0000 L CNN
-F 2 "" V 2490 7040 50  0001 C CNN
+F 2 "Resistor_THT:R_Axial_DIN0207_L6.3mm_D2.5mm_P7.62mm_Horizontal" V 2490 7040 50  0001 C CNN
 F 3 "~" H 2450 7050 50  0001 C CNN
 	1    2450 7050
@@
 F 0 "R31" H 2868 7096 50  0000 L CNN
 F 1 "220Ω" H 2868 7005 50  0000 L CNN
-F 2 "" V 2840 7040 50  0001 C CNN
+F 2 "Resistor_THT:R_Axial_DIN0207_L6.3mm_D2.5mm_P7.62mm_Horizontal" V 2840 7040 50  0001 C CNN
 F 3 "~" H 2800 7050 50  0001 C CNN
 	1    2800 7050
@@
 F 0 "R32" H 3218 7096 50  0000 L CNN
 F 1 "220Ω" H 3218 7005 50  0000 L CNN
-F 2 "" V 3190 7040 50  0001 C CNN
+F 2 "Resistor_THT:R_Axial_DIN0207_L6.3mm_D2.5mm_P7.62mm_Horizontal" V 3190 7040 50  0001 C CNN
 F 3 "~" H 3150 7050 50  0001 C CNN
 	1    3150 7050
@@
 F 0 "R33" H 3568 7096 50  0000 L CNN
 F 1 "220Ω" H 3568 7005 50  0000 L CNN
-F 2 "" V 3540 7040 50  0001 C CNN
+F 2 "Resistor_THT:R_Axial_DIN0207_L6.3mm_D2.5mm_P7.62mm_Horizontal" V 3540 7040 50  0001 C CNN
 F 3 "~" H 3500 7050 50  0001 C CNN
 	1    3500 7050
@@
 F 0 "R34" H 3918 7096 50  0000 L CNN
 F 1 "220Ω" H 3918 7005 50  0000 L CNN
-F 2 "" V 3890 7040 50  0001 C CNN
+F 2 "Resistor_THT:R_Axial_DIN0207_L6.3mm_D2.5mm_P7.62mm_Horizontal" V 3890 7040 50  0001 C CNN
 F 3 "~" H 3850 7050 50  0001 C CNN
 	1    3850 7050
@@
 F 0 "R35" H 4268 7096 50  0000 L CNN
 F 1 "220Ω" H 4268 7005 50  0000 L CNN
-F 2 "" V 4240 7040 50  0001 C CNN
+F 2 "Resistor_THT:R_Axial_DIN0207_L6.3mm_D2.5mm_P7.62mm_Horizontal" V 4240 7040 50  0001 C CNN
 F 3 "~" H 4200 7050 50  0001 C CNN
 	1    4200 7050
@@
 F 0 "R36" H 4618 7096 50  0000 L CNN
 F 1 "220Ω" H 4618 7005 50  0000 L CNN
-F 2 "" V 4590 7040 50  0001 C CNN
+F 2 "Resistor_THT:R_Axial_DIN0207_L6.3mm_D2.5mm_P7.62mm_Horizontal" V 4590 7040 50  0001 C CNN
 F 3 "~" H 4550 7050 50  0001 C CNN
 	1    4550 7050
@@
 F 0 "R37" H 4968 7096 50  0000 L CNN
 F 1 "220Ω" H 4968 7005 50  0000 L CNN
-F 2 "" V 4940 7040 50  0001 C CNN
+F 2 "Resistor_THT:R_Axial_DIN0207_L6.3mm_D2.5mm_P7.62mm_Horizontal" V 4940 7040 50  0001 C CNN
 F 3 "~" H 4900 7050 50  0001 C CNN
 	1    4900 7050
@@
 F 0 "R38" H 5318 7096 50  0000 L CNN
 F 1 "220Ω" H 5318 7005 50  0000 L CNN
-F 2 "" V 5290 7040 50  0001 C CNN
+F 2 "Resistor_THT:R_Axial_DIN0207_L6.3mm_D2.5mm_P7.62mm_Horizontal" V 5290 7040 50  0001 C CNN
 F 3 "~" H 5250 7050 50  0001 C CNN
 	1    5250 7050
@@
 F 0 "R39" H 5668 7096 50  0000 L CNN
 F 1 "220Ω" H 5668 7005 50  0000 L CNN
-F 2 "" V 5640 7040 50  0001 C CNN
+F 2 "Resistor_THT:R_Axial_DIN0207_L6.3mm_D2.5mm_P7.62mm_Horizontal" V 5640 7040 50  0001 C CNN
 F 3 "~" H 5600 7050 50  0001 C CNN
 	1    5600 7050
@@
 F 0 "R40" H 6018 7096 50  0000 L CNN
 F 1 "220Ω" H 6018 7005 50  0000 L CNN
-F 2 "" V 5990 7040 50  0001 C CNN
+F 2 "Resistor_THT:R_Axial_DIN0207_L6.3mm_D2.5mm_P7.62mm_Horizontal" V 5990 7040 50  0001 C CNN
 F 3 "~" H 5950 7050 50  0001 C CNN
 	1    5950 7050
@@
 F 0 "D25" V 739 6483 50  0000 R CNN
 F 1 "LED" V 648 6483 50  0000 R CNN
-F 2 "" H 700 6600 50  0001 C CNN
+F 2 "LED_THT:LED_D5.0mm" H 700 6600 50  0001 C CNN
 F 3 "~" H 700 6600 50  0001 C CNN
 	1    700  6600

Commit message: Assign a bunch more footprints. All are assigned now.
Parts:
- U46, U47, U49, U50: footprint (none) -> Package_DIP:DIP-16_W7.62mm
- U48, U51: footprint (none) -> Package_DIP:DIP-20_W7.62mm
Changed lines of the file:
@@
 F 0 "U46" H 1850 3000 50  0000 C CNN
 F 1 "74F157" H 1850 2900 50  0000 C CNN
-F 2 "" H 2100 2100 50  0001 C CNN
+F 2 "Package_DIP:DIP-16_W7.62mm" H 2100 2100 50  0001 C CNN
 F 3 "http://www.ti.com/lit/gpn/sn74LS157" H 2100 2100 50  0001 C CNN
 	1    2100 2100
@@
 F 0 "U48" H 4100 5400 50  0000 C CNN
 F 1 "74F574" H 4100 5300 50  0000 C CNN
-F 2 "" H 4350 4600 50  0001 C CNN
+F 2 "Package_DIP:DIP-20_W7.62mm" H 4350 4600 50  0001 C CNN
 F 3 "http://www.ti.com/lit/gpn/sn74LS574" H 4350 4600 50  0001 C CNN
 	1    4350 4600
@@
 F 0 "U51" H 8700 5400 50  0000 C CNN
 F 1 "74F574" H 8700 5300 50  0000 C CNN
-F 2 "" H 8950 4600 50  0001 C CNN
+F 2 "Package_DIP:DIP-20_W7.62mm" H 8950 4600 50  0001 C CNN
 F 3 "http://www.ti.com/lit/gpn/sn74LS574" H 8950 4600 50  0001 C CNN
 	1    8950 4600
@@
 F 0 "U47" H 4100 3000 50  0000 C CNN
 F 1 "74F157" H 4100 2900 50  0000 C CNN
-F 2 "" H 4350 2100 50  0001 C CNN
+F 2 "Package_DIP:DIP-16_W7.62mm" H 4350 2100 50  0001 C CNN
 F 3 "http://www.ti.com/lit/gpn/sn74LS157" H 4350 2100 50  0001 C CNN
 	1    4350 2100
@@
 F 0 "U49" H 6400 3000 50  0000 C CNN
 F 1 "74F157" H 6400 2900 50  0000 C CNN
-F 2 "" H 6650 2100 50  0001 C CNN
+F 2 "Package_DIP:DIP-16_W7.62mm" H 6650 2100 50  0001 C CNN
 F 3 "http://www.ti.com/lit/gpn/sn74LS157" H 6650 2100 50  0001 C CNN
 	1    6650 2100
@@
 F 0 "U50" H 8700 3000 50  0000 C CNN
 F 1 "74F157" H 8700 2900 50  0000 C CNN
-F 2 "" H 8950 2100 50  0001 C CNN
+F 2 "Package_DIP:DIP-16_W7.62mm" H 8950 2100 50  0001 C CNN
 F 3 "http://www.ti.com/lit/gpn/sn74LS157" H 8950 2100 50  0001 C CNN
 	1    8950 2100
