File: Schematics/Instruction RAM.sch (KiCad schematic (older format))
At the start: 8 parts

Commit message: annotate
Parts:
- gave numbers to parts that had none: 8
Changed lines of the file:
@@
 AR Path="/5D2C07CD/5D8D004F" Ref="C?"  Part="1"
 AR Path="/5D2C1188/5D8D004F" Ref="C?"  Part="1"
-AR Path="/5D8005AF/5D800744/5D8D004F" Ref="C?"  Part="1"
-F 0 "C?" H 965 7646 50  0000 L CNN
+AR Path="/5D8005AF/5D800744/5D8D004F" Ref="C29"  Part="1"
+F 0 "C29" H 965 7646 50  0000 L CNN
 F 1 "100nF" H 965 7555 50  0000 L CNN
 F 2 "" H 888 7450 50  0001 C CNN
@@
 AR Path="/5D2C07CD/5D8D0055" Ref="C?"  Part="1"
 AR Path="/5D2C1188/5D8D0055" Ref="C?"  Part="1"
-AR Path="/5D8005AF/5D800744/5D8D0055" Ref="C?"  Part="1"
-F 0 "C?" H 1465 7646 50  0000 L CNN
+AR Path="/5D8005AF/5D800744/5D8D0055" Ref="C30"  Part="1"
+F 0 "C30" H 1465 7646 50  0000 L CNN
 F 1 "100nF" H 1465 7555 50  0000 L CNN
 F 2 "" H 1388 7450 50  0001 C CNN
@@
 AR Path="/5D2C07CD/5D8D005B" Ref="C?"  Part="1"
 AR Path="/5D2C1188/5D8D005B" Ref="C?"  Part="1"
-AR Path="/5D8005AF/5D800744/5D8D005B" Ref="C?"  Part="1"
-F 0 "C?" H 1965 7646 50  0000 L CNN
+AR Path="/5D8005AF/5D800744/5D8D005B" Ref="C31"  Part="1"
+F 0 "C31" H 1965 7646 50  0000 L CNN
 F 1 "100nF" H 1965 7555 50  0000 L CNN
 F 2 "" H 1888 7450 50  0001 C CNN
@@
 AR Path="/5D2C07CD/5D8D0061" Ref="C?"  Part="1"
 AR Path="/5D2C1188/5D8D0061" Ref="C?"  Part="1"
-AR Path="/5D8005AF/5D800744/5D8D0061" Ref="C?"  Part="1"
-F 0 "C?" H 2465 7646 50  0000 L CNN
+AR Path="/5D8005AF/5D800744/5D8D0061" Ref="C32"  Part="1"
+F 0 "C32" H 2465 7646 50  0000 L CNN
 F 1 "100nF" H 2465 7555 50  0000 L CNN
 F 2 "" H 2388 7450 50  0001 C CNN
@@
 AR Path="/5D2C07CD/5D8D0067" Ref="#PWR?"  Part="1"
 AR Path="/5D2C1188/5D8D0067" Ref="#PWR?"  Part="1"
-AR Path="/5D8005AF/5D800744/5D8D0067" Ref="#PWR?"  Part="1"
-F 0 "#PWR?" H 850 7500 50  0001 C CNN
+AR Path="/5D8005AF/5D800744/5D8D0067" Ref="#PWR0176"  Part="1"
+F 0 "#PWR0176" H 850 7500 50  0001 C CNN
 F 1 "GND" H 855 7577 50  0000 C CNN
 F 2 "" H 850 7750 50  0001 C CNN
@@
 AR Path="/5D2C07CD/5D8D006D" Ref="#PWR?"  Part="1"
 AR Path="/5D2C1188/5D8D006D" Ref="#PWR?"  Part="1"
-AR Path="/5D8005AF/5D800744/5D8D006D" Ref="#PWR?"  Part="1"
-F 0 "#PWR?" H 850 7300 50  0001 C CNN
+AR Path="/5D8005AF/5D800744/5D8D006D" Ref="#PWR0177"  Part="1"
+F 0 "#PWR0177" H 850 7300 50  0001 C CNN
 F 1 "VCC" H 867 7623 50  0000 C CNN
 F 2 "" H 850 7450 50  0001 C CNN
@@
 Connection ~ 850  7750
 $Comp
-L power:VCC #PWR?
+L power:VCC #PWR0178
 U 1 1 5D8D3093
 P 5300 1250
-F 0 "#PWR?" H 5300 1100 50  0001 C CNN
+F 0 "#PWR0178" H 5300 1100 50  0001 C CNN
 F 1 "VCC" H 5317 1423 50  0000 C CNN
 F 2 "" H 5300 1250 50  0001 C CNN
@@
 P 5300 2100
 AR Path="/5D2C1188/5D8D099F" Ref="U?"  Part="1"
-AR Path="/5D8005AF/5D800744/5D8D099F" Ref="U?"  Part="1"
-F 0 "U?" H 5750 3050 50  0000 C CNN
+AR Path="/5D8005AF/5D800744/5D8D099F" Ref="U32"  Part="1"
+F 0 "U32" H 5750 3050 50  0000 C CNN
 F 1 "IDT71256SA12TPG" H 5750 2950 50  0000 C CNN
 F 2 "" H 5300 4100 50  0001 C CNN
@@
 $EndComp
 $Comp
-L power:VCC #PWR?
+L power:VCC #PWR0179
 U 1 1 5D8D5629
 P 7300 1550
-F 0 "#PWR?" H 7300 1400 50  0001 C CNN
+F 0 "#PWR0179" H 7300 1400 50  0001 C CNN
 F 1 "VCC" H 7317 1723 50  0000 C CNN
 F 2 "" H 7300 1550 50  0001 C CNN
@@
 $EndComp
 $Comp
-L 74xx:74LS245 U?
+L 74xx:74LS245 U34
 U 1 1 5D8D3D15
 P 7300 2350
-F 0 "U?" H 7000 3150 50  0000 C CNN
+F 0 "U34" H 7000 3150 50  0000 C CNN
 F 1 "74LS245" H 7000 3050 50  0000 C CNN
 F 2 "" H 7300 2350 50  0001 C CNN
@@
 DataBus7
 $Comp
-L power:VCC #PWR?
+L power:VCC #PWR0180
 U 1 1 5D8E2F10
 P 7300 4900
-F 0 "#PWR?" H 7300 4750 50  0001 C CNN
+F 0 "#PWR0180" H 7300 4750 50  0001 C CNN
 F 1 "VCC" H 7317 5073 50  0000 C CNN
 F 2 "" H 7300 4900 50  0001 C CNN
@@
 $EndComp
 $Comp
-L 74xx:74LS245 U?
+L 74xx:74LS245 U35
 U 1 1 5D8E2F16
 P 7300 5700
-F 0 "U?" H 7000 6500 50  0000 C CNN
+F 0 "U35" H 7000 6500 50  0000 C CNN
 F 1 "74LS245" H 7000 6400 50  0000 C CNN
 F 2 "" H 7300 5700 50  0001 C CNN
@@
 	6100 2850 6800 2850
 $Comp
-L power:GND #PWR?
+L power:GND #PWR0181
 U 1 1 5D91FAFA
 P 5800 1650
-F 0 "#PWR?" H 5800 1400 50  0001 C CNN
+F 0 "#PWR0181" H 5800 1400 50  0001 C CNN
 F 1 "GND" V 5805 1522 50  0000 R CNN
 F 2 "" H 5800 1650 50  0001 C CNN
@@
 P 5300 5450
 AR Path="/5D2C1188/5D8E2F04" Ref="U?"  Part="1"
-AR Path="/5D8005AF/5D800744/5D8E2F04" Ref="U?"  Part="1"
-F 0 "U?" H 5750 6400 50  0000 C CNN
+AR Path="/5D8005AF/5D800744/5D8E2F04" Ref="U33"  Part="1"
+F 0 "U33" H 5750 6400 50  0000 C CNN
 F 1 "IDT71256SA12TPG" H 5750 6300 50  0000 C CNN
 F 2 "" H 5300 7450 50  0001 C CNN
@@
 $EndComp
 $Comp
-L power:GND #PWR?
+L power:GND #PWR0182
 U 1 1 5D92041C
 P 5800 5000
-F 0 "#PWR?" H 5800 4750 50  0001 C CNN
+F 0 "#PWR0182" H 5800 4750 50  0001 C CNN
 F 1 "GND" V 5805 4872 50  0000 R CNN
 F 2 "" H 5800 5000 50  0001 C CNN
@@
 	6000 4800 5800 4800
 $Comp
-L power:VCC #PWR?
+L power:VCC #PWR0183
 U 1 1 5D8E2EF8
 P 5300 4600
-F 0 "#PWR?" H 5300 4450 50  0001 C CNN
+F 0 "#PWR0183" H 5300 4450 50  0001 C CNN
 F 1 "VCC" H 5317 4773 50  0000 C CNN
 F 2 "" H 5300 4600 50  0001 C CNN
@@
 AddressBus
 $Comp
-L power:GND #PWR?
+L power:GND #PWR0184
 U 1 1 5DBCC3A9
 P 7300 6500
-F 0 "#PWR?" H 7300 6250 50  0001 C CNN
+F 0 "#PWR0184" H 7300 6250 50  0001 C CNN
 F 1 "GND" H 7305 6327 50  0000 C CNN
 F 2 "" H 7300 6500 50  0001 C CNN
@@
 $EndComp
 $Comp
-L power:GND #PWR?
+L power:GND #PWR0185
 U 1 1 5DBCC424
 P 5300 6400
-F 0 "#PWR?" H 5300 6150 50  0001 C CNN
+F 0 "#PWR0185" H 5300 6150 50  0001 C CNN
 F 1 "GND" H 5305 6227 50  0000 C CNN
 F 2 "" H 5300 6400 50  0001 C CNN
@@
 $EndComp
 $Comp
-L power:GND #PWR?
+L power:GND #PWR0186
 U 1 1 5DBCCD1B
 P 7300 3150
-F 0 "#PWR?" H 7300 2900 50  0001 C CNN
+F 0 "#PWR0186" H 7300 2900 50  0001 C CNN
 F 1 "GND" H 7305 2977 50  0000 C CNN
 F 2 "" H 7300 3150 50  0001 C CNN
@@
 $EndComp
 $Comp
-L power:GND #PWR?
+L power:GND #PWR0187
 U 1 1 5DBCD74B
 P 5300 3050
-F 0 "#PWR?" H 5300 2800 50  0001 C CNN
+F 0 "#PWR0187" H 5300 2800 50  0001 C CNN
 F 1 "GND" H 5305 2877 50  0000 C CNN
 F 2 "" H 5300 3050 50  0001 C CNN

Commit message: Add footprints to all decoupling caps
Parts:
- C29, C30, C31, C32: footprint (none) -> Capacitor_THT:C_Disc_D4.3mm_W1.9mm_P5.00mm
Changed lines of the file:
@@
 F 0 "C29" H 965 7646 50  0000 L CNN
 F 1 "100nF" H 965 7555 50  0000 L CNN
-F 2 "" H 888 7450 50  0001 C CNN
+F 2 "Capacitor_THT:C_Disc_D4.3mm_W1.9mm_P5.00mm" H 888 7450 50  0001 C CNN
 F 3 "~" H 850 7600 50  0001 C CNN
 	1    850  7600
@@
 F 0 "C30" H 1465 7646 50  0000 L CNN
 F 1 "100nF" H 1465 7555 50  0000 L CNN
-F 2 "" H 1388 7450 50  0001 C CNN
+F 2 "Capacitor_THT:C_Disc_D4.3mm_W1.9mm_P5.00mm" H 1388 7450 50  0001 C CNN
 F 3 "~" H 1350 7600 50  0001 C CNN
 	1    1350 7600
@@
 F 0 "C31" H 1965 7646 50  0000 L CNN
 F 1 "100nF" H 1965 7555 50  0000 L CNN
-F 2 "" H 1888 7450 50  0001 C CNN
+F 2 "Capacitor_THT:C_Disc_D4.3mm_W1.9mm_P5.00mm" H 1888 7450 50  0001 C CNN
 F 3 "~" H 1850 7600 50  0001 C CNN
 	1    1850 7600
@@
 F 0 "C32" H 2465 7646 50  0000 L CNN
 F 1 "100nF" H 2465 7555 50  0000 L CNN
-F 2 "" H 2388 7450 50  0001 C CNN
+F 2 "Capacitor_THT:C_Disc_D4.3mm_W1.9mm_P5.00mm" H 2388 7450 50  0001 C CNN
 F 3 "~" H 2350 7600 50  0001 C CNN
 	1    2350 7600

Commit message: Assign a bunch more footprints. All are assigned now.
Parts:
- U32, U33: footprint (none) -> Package_DIP:DIP-28_W7.62mm_Socket
- U34, U35: footprint (none) -> Package_DIP:DIP-20_W7.62mm_Socket
Changed lines of the file:
@@
 F 0 "U32" H 5750 3050 50  0000 C CNN
 F 1 "IDT71256SA12TPG" H 5750 2950 50  0000 C CNN
-F 2 "" H 5300 4100 50  0001 C CNN
+F 2 "Package_DIP:DIP-28_W7.62mm_Socket" H 5300 4100 50  0001 C CNN
 F 3 "" H 5300 4100 50  0001 C CNN
 	1    5300 2100
@@
 F 0 "U34" H 7000 3150 50  0000 C CNN
 F 1 "74LS245" H 7000 3050 50  0000 C CNN
-F 2 "" H 7300 2350 50  0001 C CNN
+F 2 "Package_DIP:DIP-20_W7.62mm_Socket" H 7300 2350 50  0001 C CNN
 F 3 "http://www.ti.com/lit/gpn/sn74LS245" H 7300 2350 50  0001 C CNN
 	1    7300 2350
@@
 F 0 "U35" H 7000 6500 50  0000 C CNN
 F 1 "74LS245" H 7000 6400 50  0000 C CNN
-F 2 "" H 7300 5700 50  0001 C CNN
+F 2 "Package_DIP:DIP-20_W7.62mm_Socket" H 7300 5700 50  0001 C CNN
 F 3 "http://www.ti.com/lit/gpn/sn74LS245" H 7300 5700 50  0001 C CNN
 	1    7300 5700
@@
 F 0 "U33" H 5750 6400 50  0000 C CNN
 F 1 "IDT71256SA12TPG" H 5750 6300 50  0000 C CNN
-F 2 "" H 5300 7450 50  0001 C CNN
+F 2 "Package_DIP:DIP-28_W7.62mm_Socket" H 5300 7450 50  0001 C CNN
 F 3 "" H 5300 7450 50  0001 C CNN
 	1    5300 5450

Commit message: My buses were not named according the rules in the Eeschema manual.
Buses which connect to global labels must be named specially.
Connections:
- net AddressBus00 renamed AddressBus0
- net AddressBus01 renamed AddressBus1
- net AddressBus02 renamed AddressBus2
- net AddressBus03 renamed AddressBus3
- net AddressBus04 renamed AddressBus4
- net AddressBus05 renamed AddressBus5
- net AddressBus06 renamed AddressBus6
- net AddressBus07 renamed AddressBus7
- net AddressBus08 renamed AddressBus8
- net AddressBus09 renamed AddressBus9
- net IRAM00 renamed IRAM0
- net IRAM01 renamed IRAM1
- net IRAM02 renamed IRAM2
- net IRAM03 renamed IRAM3
- net IRAM04 renamed IRAM4
- net IRAM05 renamed IRAM5
- net IRAM06 renamed IRAM6
- net IRAM07 renamed IRAM7
- net IRAM08 renamed IRAM8
- net IRAM09 renamed IRAM9
Changed lines of the file:
@@
 	8300 5100 8200 5200
 Wire Bus Line
-	8300 3450 10000 3450
-Text GLabel 10000 3450 2    50   Output ~ 0
-DataBus
+	8300 3450 9900 3450
+Text GLabel 9900 3450 2    50   Output ~ 0
+DataBus[0..7]
 Entry Wire Line
 	6200 1850 6300 1950
@@
 Entry Wire Line
 	6200 2550 6300 2650
-Text GLabel 10000 3600 2    50   Output ~ 0
-IRAM
-Wire Bus Line
-	10000 3600 6300 3600
+Text GLabel 9900 3600 2    50   Output ~ 0
+IRAM[0..15]
+Wire Bus Line
+	9900 3600 6300 3600
 Entry Wire Line
 	6200 5300 6300 5200
@@
 	6200 5800 6300 5700
 Text Label 6650 5200 2    50   ~ 0
-IRAM00
+IRAM0
 Text Label 6650 5300 2    50   ~ 0
-IRAM01
+IRAM1
 Text Label 6650 5400 2    50   ~ 0
-IRAM02
+IRAM2
 Text Label 6650 5500 2    50   ~ 0
-IRAM03
+IRAM3
 Text Label 6650 5600 2    50   ~ 0
-IRAM04
+IRAM4
 Text Label 6650 5700 2    50   ~ 0
-IRAM05
+IRAM5
 Text Label 6650 5800 2    50   ~ 0
-IRAM06
+IRAM6
 Text Label 6650 5900 2    50   ~ 0
-IRAM07
+IRAM7
 Text Label 6650 1850 2    50   ~ 0
-IRAM08
+IRAM8
 Text Label 6650 1950 2    50   ~ 0
-IRAM09
+IRAM9
 Text Label 6650 2050 2    50   ~ 0
 IRAM10
@@
 Text Label 6650 2550 2    50   ~ 0
 IRAM15
-Text GLabel 1050 2450 0    50   Input ~ 0
-DeviceSelect
+Text GLabel 1250 2450 0    50   Input ~ 0
+DeviceSelect[0..7]
 Text Label 1400 2250 0    50   ~ 0
 DeviceSelect3
@@
 	6100 6200 6100 4000
 Wire Bus Line
-	1300 2450 1050 2450
+	1300 2450 1250 2450
 Connection ~ 1300 2450
 Wire Bus Line
@@
 	4200 1450 4800 1450
 Text Label 4750 1450 2    50   ~ 0
-AddressBus00
+AddressBus0
 Entry Wire Line
 	4200 1550 4100 1650
@@
 	4200 1550 4800 1550
 Text Label 4750 1550 2    50   ~ 0
-AddressBus01
+AddressBus1
 Entry Wire Line
 	4200 1650 4100 1750
@@
 	4200 1650 4800 1650
 Text Label 4750 1650 2    50   ~ 0
-AddressBus02
+AddressBus2
 Entry Wire Line
 	4200 1750 4100 1850
@@
 	4200 1750 4800 1750
 Text Label 4750 1750 2    50   ~ 0
-AddressBus03
+AddressBus3
 Entry Wire Line
 	4200 1850 4100 1950
@@
 	4200 1850 4800 1850
 Text Label 4750 1850 2    50   ~ 0
-AddressBus04
+AddressBus4
 Entry Wire Line
 	4200 1950 4100 2050
@@
 	4200 1950 4800 1950
 Text Label 4750 1950 2    50   ~ 0
-AddressBus05
+AddressBus5
 Entry Wire Line
 	4200 2050 4100 2150
@@
 	4200 2050 4800 2050
 Text Label 4750 2050 2    50   ~ 0
-AddressBus06
+AddressBus6
 Entry Wire Line
 	4200 2150 4100 2250
@@
 	4200 2150 4800 2150
 Text Label 4750 2150 2    50   ~ 0
-AddressBus07
+AddressBus7
 Entry Wire Line
 	4200 2250 4100 2350
@@
 	4200 2250 4800 2250
 Text Label 4750 2250 2    50   ~ 0
-AddressBus08
+AddressBus8
 Entry Wire Line
 	4200 2350 4100 2450
@@
 	4200 2350 4800 2350
 Text Label 4750 2350 2    50   ~ 0
-AddressBus09
+AddressBus9
 Entry Wire Line
 	4200 2450 4100 2550
@@
 	4200 4800 4800 4800
 Text Label 4750 4800 2    50   ~ 0
-AddressBus00
+AddressBus0
 Entry Wire Line
 	4200 4900 4100 5000
@@
 	4200 4900 4800 4900
 Text Label 4750 4900 2    50   ~ 0
-AddressBus01
+AddressBus1
 Entry Wire Line
 	4200 5000 4100 5100
@@
 	4200 5000 4800 5000
 Text Label 4750 5000 2    50   ~ 0
-AddressBus02
+AddressBus2
 Entry Wire Line
 	4200 5100 4100 5200
@@
 	4200 5100 4800 5100
 Text Label 4750 5100 2    50   ~ 0
-AddressBus03
+AddressBus3
 Entry Wire Line
 	4200 5200 4100 5300
@@
 	4200 5200 4800 5200
 Text Label 4750 5200 2    50   ~ 0
-AddressBus04
+AddressBus4
 Entry Wire Line
 	4200 5300 4100 5400
@@
 	4200 5300 4800 5300
 Text Label 4750 5300 2    50   ~ 0
-AddressBus05
+AddressBus5
 Entry Wire Line
 	4200 5400 4100 5500
@@
 	4200 5400 4800 5400
 Text Label 4750 5400 2    50   ~ 0
-AddressBus06
+AddressBus6
 Entry Wire Line
 	4200 5500 4100 5600
@@
 	4200 5500 4800 5500
 Text Label 4750 5500 2    50   ~ 0
-AddressBus07
+AddressBus7
 Entry Wire Line
 	4200 5600 4100 5700
@@
 	4200 5600 4800 5600
 Text Label 4750 5600 2    50   ~ 0
-AddressBus08
+AddressBus8
 Entry Wire Line
 	4200 5700 4100 5800
@@
 	4200 5700 4800 5700
 Text Label 4750 5700 2    50   ~ 0
-AddressBus09
+AddressBus9
 Entry Wire Line
 	4200 5800 4100 5900
@@
 AddressBus14
 Wire Bus Line
-	4100 6500 1050 6500
-Text GLabel 1050 6500 0    50   Input ~ 0
-AddressBus
+	4100 6500 1250 6500
+Text GLabel 1250 6500 0    50   Input ~ 0
+AddressBus[0..15]
 $Comp
 L power:GND #PWR0184
@@
 Wire Wire Line
 	6100 4000 3700 4000
+Wire Bus Line
+	6300 1950 6300 3600
+Wire Bus Line
+	6300 3600 6300 5800
 Wire Wire Line
 	5800 5900 6800 5900
@@
 	5800 5700 6800 5700
 Wire Bus Line
-	6300 1950 6300 3600
-Wire Bus Line
-	6300 3600 6300 5800
-Wire Bus Line
 	8300 3450 8300 5800

Commit message: Add unused IC units to Output Display to ensure no ICs are shared with other modules.
Parts:
- renumbered U32 to U31, U33 to U32, U34 to U33, U35 to U34
Changed lines of the file:
@@
 AR Path="/5D2C07CD/5D8D0067" Ref="#PWR?"  Part="1"
 AR Path="/5D2C1188/5D8D0067" Ref="#PWR?"  Part="1"
-AR Path="/5D8005AF/5D800744/5D8D0067" Ref="#PWR0176"  Part="1"
-F 0 "#PWR0176" H 850 7500 50  0001 C CNN
+AR Path="/5D8005AF/5D800744/5D8D0067" Ref="#PWR077"  Part="1"
+F 0 "#PWR077" H 850 7500 50  0001 C CNN
 F 1 "GND" H 855 7577 50  0000 C CNN
 F 2 "" H 850 7750 50  0001 C CNN
@@
 AR Path="/5D2C07CD/5D8D006D" Ref="#PWR?"  Part="1"
 AR Path="/5D2C1188/5D8D006D" Ref="#PWR?"  Part="1"
-AR Path="/5D8005AF/5D800744/5D8D006D" Ref="#PWR0177"  Part="1"
-F 0 "#PWR0177" H 850 7300 50  0001 C CNN
+AR Path="/5D8005AF/5D800744/5D8D006D" Ref="#PWR076"  Part="1"
+F 0 "#PWR076" H 850 7300 50  0001 C CNN
 F 1 "VCC" H 867 7623 50  0000 C CNN
 F 2 "" H 850 7450 50  0001 C CNN
@@
 Connection ~ 850  7750
 $Comp
-L power:VCC #PWR0178
+L power:VCC #PWR078
 U 1 1 5D8D3093
 P 5300 1250
-F 0 "#PWR0178" H 5300 1100 50  0001 C CNN
+F 0 "#PWR078" H 5300 1100 50  0001 C CNN
 F 1 "VCC" H 5317 1423 50  0000 C CNN
 F 2 "" H 5300 1250 50  0001 C CNN
@@
 P 5300 2100
 AR Path="/5D2C1188/5D8D099F" Ref="U?"  Part="1"
-AR Path="/5D8005AF/5D800744/5D8D099F" Ref="U32"  Part="1"
-F 0 "U32" H 5750 3050 50  0000 C CNN
+AR Path="/5D8005AF/5D800744/5D8D099F" Ref="U31"  Part="1"
+F 0 "U31" H 5750 3050 50  0000 C CNN
 F 1 "IDT71256SA12TPG" H 5750 2950 50  0000 C CNN
 F 2 "Package_DIP:DIP-28_W7.62mm_Socket" H 5300 4100 50  0001 C CNN
@@
 $EndComp
 $Comp
-L power:VCC #PWR0179
+L power:VCC #PWR084
 U 1 1 5D8D5629
 P 7300 1550
-F 0 "#PWR0179" H 7300 1400 50  0001 C CNN
+F 0 "#PWR084" H 7300 1400 50  0001 C CNN
 F 1 "VCC" H 7317 1723 50  0000 C CNN
 F 2 "" H 7300 1550 50  0001 C CNN
@@
 $EndComp
 $Comp
-L 74xx:74LS245 U34
+L 74xx:74LS245 U33
 U 1 1 5D8D3D15
 P 7300 2350
-F 0 "U34" H 7000 3150 50  0000 C CNN
+F 0 "U33" H 7000 3150 50  0000 C CNN
 F 1 "74LS245" H 7000 3050 50  0000 C CNN
 F 2 "Package_DIP:DIP-20_W7.62mm_Socket" H 7300 2350 50  0001 C CNN
@@
 DataBus7
 $Comp
-L power:VCC #PWR0180
+L power:VCC #PWR086
 U 1 1 5D8E2F10
 P 7300 4900
-F 0 "#PWR0180" H 7300 4750 50  0001 C CNN
+F 0 "#PWR086" H 7300 4750 50  0001 C CNN
 F 1 "VCC" H 7317 5073 50  0000 C CNN
 F 2 "" H 7300 4900 50  0001 C CNN
@@
 $EndComp
 $Comp
-L 74xx:74LS245 U35
+L 74xx:74LS245 U34
 U 1 1 5D8E2F16
 P 7300 5700
-F 0 "U35" H 7000 6500 50  0000 C CNN
+F 0 "U34" H 7000 6500 50  0000 C CNN
 F 1 "74LS245" H 7000 6400 50  0000 C CNN
 F 2 "Package_DIP:DIP-20_W7.62mm_Socket" H 7300 5700 50  0001 C CNN
@@
 	6100 2850 6800 2850
 $Comp
-L power:GND #PWR0181
+L power:GND #PWR082
 U 1 1 5D91FAFA
 P 5800 1650
-F 0 "#PWR0181" H 5800 1400 50  0001 C CNN
+F 0 "#PWR082" H 5800 1400 50  0001 C CNN
 F 1 "GND" V 5805 1522 50  0000 R CNN
 F 2 "" H 5800 1650 50  0001 C CNN
@@
 P 5300 5450
 AR Path="/5D2C1188/5D8E2F04" Ref="U?"  Part="1"
-AR Path="/5D8005AF/5D800744/5D8E2F04" Ref="U33"  Part="1"
-F 0 "U33" H 5750 6400 50  0000 C CNN
+AR Path="/5D8005AF/5D800744/5D8E2F04" Ref="U32"  Part="1"
+F 0 "U32" H 5750 6400 50  0000 C CNN
 F 1 "IDT71256SA12TPG" H 5750 6300 50  0000 C CNN
 F 2 "Package_DIP:DIP-28_W7.62mm_Socket" H 5300 7450 50  0001 C CNN
@@
 $EndComp
 $Comp
-L power:GND #PWR0182
+L power:GND #PWR083
 U 1 1 5D92041C
 P 5800 5000
-F 0 "#PWR0182" H 5800 4750 50  0001 C CNN
+F 0 "#PWR083" H 5800 4750 50  0001 C CNN
 F 1 "GND" V 5805 4872 50  0000 R CNN
 F 2 "" H 5800 5000 50  0001 C CNN
@@
 	6000 4800 5800 4800
 $Comp
-L power:VCC #PWR0183
+L power:VCC #PWR080
 U 1 1 5D8E2EF8
 P 5300 4600
-F 0 "#PWR0183" H 5300 4450 50  0001 C CNN
+F 0 "#PWR080" H 5300 4450 50  0001 C CNN
 F 1 "VCC" H 5317 4773 50  0000 C CNN
 F 2 "" H 5300 4600 50  0001 C CNN
@@
 AddressBus[0..15]
 $Comp
-L power:GND #PWR0184
+L power:GND #PWR087
 U 1 1 5DBCC3A9
 P 7300 6500
-F 0 "#PWR0184" H 7300 6250 50  0001 C CNN
+F 0 "#PWR087" H 7300 6250 50  0001 C CNN
 F 1 "GND" H 7305 6327 50  0000 C CNN
 F 2 "" H 7300 6500 50  0001 C CNN
@@
 $EndComp
 $Comp
-L power:GND #PWR0185
+L power:GND #PWR081
 U 1 1 5DBCC424
 P 5300 6400
-F 0 "#PWR0185" H 5300 6150 50  0001 C CNN
+F 0 "#PWR081" H 5300 6150 50  0001 C CNN
 F 1 "GND" H 5305 6227 50  0000 C CNN
 F 2 "" H 5300 6400 50  0001 C CNN
@@
 $EndComp
 $Comp
-L power:GND #PWR0186
+L power:GND #PWR085
 U 1 1 5DBCCD1B
 P 7300 3150
-F 0 "#PWR0186" H 7300 2900 50  0001 C CNN
+F 0 "#PWR085" H 7300 2900 50  0001 C CNN
 F 1 "GND" H 7305 2977 50  0000 C CNN
 F 2 "" H 7300 3150 50  0001 C CNN
@@
 $EndComp
 $Comp
-L power:GND #PWR0187
+L power:GND #PWR079
 U 1 1 5DBCD74B
 P 5300 3050
-F 0 "#PWR0187" H 5300 2800 50  0001 C CNN
+F 0 "#PWR079" H 5300 2800 50  0001 C CNN
 F 1 "GND" H 5305 2877 50  0000 C CNN
 F 2 "" H 5300 3050 50  0001 C CNN

Commit message: Add unused IC units to Data RAM to ensure no ICs are shared with other modules.
Parts:
- renumbered U31 to U30, U32 to U31, U33 to U32, U34 to U33
Changed lines of the file:
@@
 P 5300 2100
 AR Path="/5D2C1188/5D8D099F" Ref="U?"  Part="1"
-AR Path="/5D8005AF/5D800744/5D8D099F" Ref="U31"  Part="1"
-F 0 "U31" H 5750 3050 50  0000 C CNN
+AR Path="/5D8005AF/5D800744/5D8D099F" Ref="U30"  Part="1"
+F 0 "U30" H 5750 3050 50  0000 C CNN
 F 1 "IDT71256SA12TPG" H 5750 2950 50  0000 C CNN
 F 2 "Package_DIP:DIP-28_W7.62mm_Socket" H 5300 4100 50  0001 C CNN
@@
 $EndComp
 $Comp
-L 74xx:74LS245 U33
+L 74xx:74LS245 U32
 U 1 1 5D8D3D15
 P 7300 2350
-F 0 "U33" H 7000 3150 50  0000 C CNN
+F 0 "U32" H 7000 3150 50  0000 C CNN
 F 1 "74LS245" H 7000 3050 50  0000 C CNN
 F 2 "Package_DIP:DIP-20_W7.62mm_Socket" H 7300 2350 50  0001 C CNN
@@
 $EndComp
 $Comp
-L 74xx:74LS245 U34
+L 74xx:74LS245 U33
 U 1 1 5D8E2F16
 P 7300 5700
-F 0 "U34" H 7000 6500 50  0000 C CNN
+F 0 "U33" H 7000 6500 50  0000 C CNN
 F 1 "74LS245" H 7000 6400 50  0000 C CNN
 F 2 "Package_DIP:DIP-20_W7.62mm_Socket" H 7300 5700 50  0001 C CNN
@@
 P 5300 5450
 AR Path="/5D2C1188/5D8E2F04" Ref="U?"  Part="1"
-AR Path="/5D8005AF/5D800744/5D8E2F04" Ref="U32"  Part="1"
-F 0 "U32" H 5750 6400 50  0000 C CNN
+AR Path="/5D8005AF/5D800744/5D8E2F04" Ref="U31"  Part="1"
+F 0 "U31" H 5750 6400 50  0000 C CNN
 F 1 "IDT71256SA12TPG" H 5750 6300 50  0000 C CNN
 F 2 "Package_DIP:DIP-28_W7.62mm_Socket" H 5300 7450 50  0001 C CNN

Commit message: Change assignment of logic units to reduce the number of discrete ICs.
This reduces part count in the Instruction RAM module.
Parts:
- added C33, C34, C35: 100nF, Capacitor_THT:C_Disc_D4.3mm_W1.9mm_P5.00mm, symbol Device:C
- added U34, U37: 74LS08, Package_DIP:DIP-14_W7.62mm, symbol 74xx:74LS08
- added U35: 74LS04, Package_DIP:DIP-14_W7.62mm, symbol 74xx:74LS04
- added U36, U39: 74LS32, Package_DIP:DIP-14_W7.62mm, symbol 74xx:74LS32
Connections:
- net DeviceSelect3: now also U35.1, U36.2, U39.2
- net DeviceSelect4: now also U35.3, U36.10, U36.13
- net GND: now also C33.2, C34.2, C35.2
- net VCC: now also C33.1, C34.1, C35.1
- net ~MI: now also U34.1, U34.12, U36.12, U39.1
- net Lower Instruction RAM Control/~OE: no longer names the net of U31.22 (~OE)
- net Lower Instruction RAM Control/~OE: now also U34.8
- net Lower Instruction RAM Control/~OutToBus: no longer names the net of U33.19 (CE)
- net Lower Instruction RAM Control/~OutToBus: now also U36.8
- net Lower Instruction RAM Control/~WE: no longer names the net of U31.27 (~WE)
- net Lower Instruction RAM Control/~WE: now also U36.11
- net Upper Instruction RAM Control/~OE: no longer names the net of U30.22 (~OE)
- net Upper Instruction RAM Control/~OE: now also U37.3
- net Upper Instruction RAM Control/~OutToBus: no longer names the net of U32.19 (CE)
- net Upper Instruction RAM Control/~OutToBus: now also U36.3
- net Upper Instruction RAM Control/~WE: no longer names the net of U30.27 (~WE)
- net Upper Instruction RAM Control/~WE: now also U39.3
- new net: U35.2, U37.1
- new net: U34.3, U36.1
- new net: U34.9, U35.4
- new net: U34.11, U36.9
- new net ~MO: U34.10, U34.13, U34.2, U37.2
- no-connect marks 0 -> 8
