File: Schematics/Serial.sch (KiCad schematic (older format))
At the start: 1 part

Commit message: annotate
Parts:
- gave numbers to parts that had none: 1
Changed lines of the file:
@@
 $EndDescr
 $Comp
-L MCU_Module:Arduino_Nano_v3.x A?
+L MCU_Module:Arduino_Nano_v3.x A1
 U 1 1 5D7E59B1
 P 6150 4000
-F 0 "A?" H 5550 5100 50  0000 C CNN
+F 0 "A1" H 5550 5100 50  0000 C CNN
 F 1 "Arduino_Nano_v3.x" H 5600 5000 50  0000 C CNN
 F 2 "Module:Arduino_Nano" H 6300 3050 50  0001 L CNN
@@
 $EndComp
 $Comp
-L power:VCC #PWR?
+L power:VCC #PWR0122
 U 1 1 5D7E6F02
 P 6050 3000
-F 0 "#PWR?" H 6050 2850 50  0001 C CNN
+F 0 "#PWR0122" H 6050 2850 50  0001 C CNN
 F 1 "VCC" H 6067 3173 50  0000 C CNN
 F 2 "" H 6050 3000 50  0001 C CNN
@@
 NoConn ~ 6350 3000
 $Comp
-L power:GND #PWR?
+L power:GND #PWR0123
 U 1 1 5D7E7F51
 P 6200 5100
-F 0 "#PWR?" H 6200 4850 50  0001 C CNN
+F 0 "#PWR0123" H 6200 4850 50  0001 C CNN
 F 1 "GND" H 6205 4927 50  0000 C CNN
 F 2 "" H 6200 5100 50  0001 C CNN

Commit message: My buses were not named according the rules in the Eeschema manual.
Buses which connect to global labels must be named specially.
Connections:
- net AddressBus00 renamed AddressBus0
Changed lines of the file:
@@
 ~MI
 Text GLabel 4050 4800 0    50   Input ~ 0
-AddressBus
+AddressBus[0..15]
 Wire Bus Line
 	4050 4800 4850 4800
@@
 	4950 4700 5650 4700
 Text Label 5000 4700 0    50   ~ 0
-AddressBus00
+AddressBus0
 Text GLabel 4050 4600 0    50   BiDi ~ 0
-DataBus
+DataBus[0..7]
 Wire Wire Line
 	5650 3600 4350 3600
