File: Schematics/Version2/MainBoard/Shifter.sch (KiCad schematic (older format))
At the start: 1 part, among them J13 Shifter Connector

Commit message: Merge branch "version2a"
This replaces the Version2 schematics with a new second version. This one
completes a four layer routing of the main board.
Connections:
- net ~ShifterOut: now reaches J13.73 (Pin_73)
- no-connect marks 5 -> 4
Other:
- note removed: "TODO: Need a control signal for Shifter output"
Changed lines of the file:
@@
 $Descr A4 11693 8268
 encoding utf-8
-Sheet 22 22
+Sheet 20 23
 Title ""
 Date ""
@@
 Wire Wire Line
 	5600 5850 5600 6200
-NoConn ~ 5050 2350
-Text Notes 3550 2250 0    50   ~ 0
-TODO: Need a control signal for Shifter output
 NoConn ~ 7150 2250
 NoConn ~ 7150 2450
 NoConn ~ 7150 2650
 NoConn ~ 5050 2550
+Text GLabel 5050 2350 0    50   Input ~ 0
+~ShifterOut
 Wire Bus Line
 	7100 2950 7100 3550
