File: Schematics/Version2/MainBoard/Execute.sch (KiCad schematic (older format))
At the start: 3 parts, among them J5 C Register LED Connector, U48 74LS245

Commit message: Merge branch "version2a"
This replaces the Version2 schematics with a new second version. This one
completes a four layer routing of the main board.
Parts:
- U48: value 74LS245 -> 74AHCT245
Other:
- note removed: "There are\nunused control\nsignals here\nfor future\nexpansion."
Changed lines of the file:
@@
 $Descr A 11000 8500
 encoding utf-8
-Sheet 11 22
+Sheet 22 23
 Title "Execute"
 Date ""
@@
 AR Path="/5D2C13FD/5D9156B5" Ref="U48"  Part="1"
 F 0 "U48" H 6450 3000 50  0000 C CNN
-F 1 "74LS245" H 6450 2900 50  0000 C CNN
+F 1 "74AHCT245" H 6450 2900 50  0000 C CNN
 F 2 "Package_DIP:DIP-20_W7.62mm" H 6750 2200 50  0001 C CNN
-F 3 "http://www.ti.com/lit/gpn/sn74LS245" H 6750 2200 50  0001 C CNN
+F 3 "http://www.ti.com/lit/ds/symlink/sn54ahct245.pdf" H 6750 2200 50  0001 C CNN
 	1    6750 2200
 	1    0    0    -1
@@
 	1    0    0    -1
 $EndComp
-Text Notes 3900 4250 0    50   ~ 0
-There are\nunused control\nsignals here\nfor future\nexpansion.
+Entry Wire Line
+	4300 4550 4400 4450
+Wire Wire Line
+	4400 3800 4400 4450
+Text Label 4400 4400 1    50   ~ 0
+ControlWord27
+Text GLabel 4400 3800 1    50   Output ~ 0
+~ShifterOut
+Entry Wire Line
+	4150 4550 4250 4450
+Wire Wire Line
+	4250 3800 4250 4450
+Text Label 4250 4400 1    50   ~ 0
+ControlWord28
+Text GLabel 4250 3800 1    50   Output ~ 0
+~KI
+Entry Wire Line
+	4000 4550 4100 4450
+Wire Wire Line
+	4100 3800 4100 4450
+Text Label 4100 4400 1    50   ~ 0
+ControlWord29
+Text GLabel 4100 3800 1    50   Output ~ 0
+~KO
 Wire Bus Line
 	1100 1050 5850 1050

Commit message: Merge branch "version2b".
This is a new version of the computer which incorporates a number of
improvements:
  * Uses a four layer PCB instead of six.
  * Replaced the clock with a new circuit. This is simpler, but allows for
    an external clock to be attached.
  * Changes to the ALU to have it operate over two clock cycles instead of
    one. This fixes a timing issue which makes the ALU unreliable at 10MHz.
  * Replaced instruction RAM with dual port SRAM.
  * Replaced the physical connector for expansion cards to interleave
    signals with ground.
  * Added places where components can be attached to provide AC termination
    of the data bus, should this be necessary.
Changed lines of the file:
@@
 $Descr A 11000 8500
 encoding utf-8
-Sheet 22 23
+Sheet 19 21
 Title "Execute"
 Date ""
@@
 	1    0    0    -1
 $EndComp
-Entry Wire Line
-	4300 4550 4400 4450
-Wire Wire Line
-	4400 3800 4400 4450
-Text Label 4400 4400 1    50   ~ 0
-ControlWord27
-Text GLabel 4400 3800 1    50   Output ~ 0
-~ShifterOut
-Entry Wire Line
-	4150 4550 4250 4450
-Wire Wire Line
-	4250 3800 4250 4450
-Text Label 4250 4400 1    50   ~ 0
-ControlWord28
-Text GLabel 4250 3800 1    50   Output ~ 0
-~KI
-Entry Wire Line
-	4000 4550 4100 4450
-Wire Wire Line
-	4100 3800 4100 4450
-Text Label 4100 4400 1    50   ~ 0
-ControlWord29
-Text GLabel 4100 3800 1    50   Output ~ 0
-~KO
 Wire Bus Line
 	1100 1050 5850 1050
