File: Schematics/Version2/MainBoard/Instruction Decode.sch (KiCad schematic (older format))
At the start: 4 parts, among them J14 Microcode ROM Connector 1, J15 Microcode ROM Connector 2, U47 74F574

Commit message: Merge branch "version2a"
This replaces the Version2 schematics with a new second version. This one
completes a four layer routing of the main board.
Parts:
- removed J14: Microcode ROM Connector 1, Connector_PinSocket_2.54mm:PinSocket_2x40_P2.54mm_Vertical, symbol Connector_Generic:Conn_02x40_Odd_Even
- removed J15: Microcode ROM Connector 2, Connector_PinSocket_2.54mm:PinSocket_2x20_P2.54mm_Vertical, symbol Connector_Generic:Conn_02x20_Odd_Even
- added C11, C24, C25, C26, C27, C4, C5, C6: 100nF, Capacitor_THT:C_Disc_D4.3mm_W1.9mm_P5.00mm, symbol Device:C
- added J14: Control Word LED Connector [16..23], Connector_PinSocket_2.54mm:PinSocket_1x09_P2.54mm_Vertical, symbol Connector:Conn_01x09_Female
- added J15: Control Word LED Connector [8..15], Connector_PinSocket_2.54mm:PinSocket_1x09_P2.54mm_Vertical, symbol Connector:Conn_01x09_Female
- added J22: Control Word LED Connector [0..7], Connector_PinSocket_2.54mm:PinSocket_1x09_P2.54mm_Vertical, symbol Connector:Conn_01x09_Female
- added J7: Control Word LED Connector [24..31], Connector_PinSocket_2.54mm:PinSocket_1x09_P2.54mm_Vertical, symbol Connector:Conn_01x09_Female
- added U16, U17, U24, U5: GLS29EE010, Package_DIP:DIP-32_W15.24mm_Socket, symbol Memory_EEPROM:GLS29EE010
- added U25, U26, U27, U28: 74AHCT574, Package_DIP:DIP-20_W7.62mm, symbol 74xx:74LS574
- U47: value 74F574 -> 74AHCT574
Connections:
- net ControlClock: now also U25.11 (Cp), U26.11 (Cp), U27.11 (Cp), U28.11 (Cp)
- net ControlWord0: now also J22.2 (Pin_2), U28.19 (Q0)
- net ControlWord1: now also J22.3 (Pin_3), U28.18 (Q1)
- net ControlWord10: now also J15.4 (Pin_4), U27.17 (Q2)
- net ControlWord11: now also J15.5 (Pin_5), U27.16 (Q3)
- net ControlWord12: now also J15.6 (Pin_6), U27.15 (Q4)
- net ControlWord13: now also J15.7 (Pin_7), U27.14 (Q5)
- net ControlWord14: now also J15.8 (Pin_8), U27.13 (Q6)
- net ControlWord15: now also J15.9 (Pin_9), U27.12 (Q7)
- net ControlWord16: now also J14.2 (Pin_2), U26.19 (Q0)
- net ControlWord17: now also J14.3 (Pin_3), U26.18 (Q1)
- net ControlWord18: now also J14.4 (Pin_4), U26.17 (Q2)
- net ControlWord19: now also J14.5 (Pin_5), U26.16 (Q3)
- net ControlWord2: now also J22.4 (Pin_4), U28.17 (Q2)
- net ControlWord20: now also J14.6 (Pin_6), U26.15 (Q4)
- net ControlWord21: now also J14.7 (Pin_7), U26.14 (Q5)
- net ControlWord22: now also J14.8 (Pin_8), U26.13 (Q6)
- net ControlWord23: now also J14.9 (Pin_9), U26.12 (Q7)
- net ControlWord24: now also J7.2 (Pin_2), U25.19 (Q0)
- net ControlWord25: now also J7.3 (Pin_3), U25.18 (Q1)
- net ControlWord26: now also J7.4 (Pin_4), U25.17 (Q2)
- net ControlWord27: now also J7.5 (Pin_5), U25.16 (Q3)
- net ControlWord28: now also J7.6 (Pin_6), U25.15 (Q4)
- net ControlWord29: now also J7.7 (Pin_7), U25.14 (Q5)
- net ControlWord3: now also J22.5 (Pin_5), U28.16 (Q3)
- net ControlWord30: now also J7.8 (Pin_8), U25.13 (Q6)
- net ControlWord31: now also J7.9 (Pin_9), U25.12 (Q7)
- net ControlWord4: now also J22.6 (Pin_6), U28.15 (Q4)
- net ControlWord5: now also J22.7 (Pin_7), U28.14 (Q5)
- net ControlWord6: now also J22.8 (Pin_8), U28.13 (Q6)
- net ControlWord7: now also J22.9 (Pin_9), U28.12 (Q7)
- net ControlWord8: now also J15.2 (Pin_2), U27.19 (Q0)
- net ControlWord9: now also J15.3 (Pin_3), U27.18 (Q1)
- net GND: now also C11.2, C24.2, C25.2, C26.2, C27.2, C4.2, C5.2, C6.2, J14.1 (Pin_1), J15.1 (Pin_1), J22.1 (Pin_1), J7.1 (Pin_1), U16.16 (VSS), U16.2 (A16), U16.22 (CE), U16.23 (A10), U16.24 (OE), U16.25 (A11), U16.28 (A13), U16.29 (A14), U16.3 (A15), U16.4 (A12), U17.16 (VSS), U17.2 (A16), U17.22 (CE), U17.23 (A10), U17.24 (OE), U17.25 (A11), U17.28 (A13), U17.29 (A14), U17.3 (A15), U17.4 (A12), U24.16 (VSS), U24.2 (A16), U24.22 (CE), U24.23 (A10), U24.24 (OE), U24.25 (A11), U24.28 (A13), U24.29 (A14), U24.3 (A15), U24.4 (A12), U25.1 (OE), U25.10 (GND), U26.1 (OE), U26.10 (GND), U27.1 (OE), U27.10 (GND), U28.1 (OE), U28.10 (GND), U5.16 (VSS), U5.2 (A16), U5.22 (CE), U5.23 (A10), U5.24 (OE), U5.25 (A11), U5.28 (A13), U5.29 (A14), U5.3 (A15), U5.4 (A12)
- net IR10: now also U16.10 (A2), U17.10 (A2), U24.10 (A2), U5.10 (A2)
- net IR11: now also U16.9 (A3), U17.9 (A3), U24.9 (A3), U5.9 (A3)
- net IR12: now also U16.8 (A4), U17.8 (A4), U24.8 (A4), U5.8 (A4)
- net IR13: now also U16.7 (A5), U17.7 (A5), U24.7 (A5), U5.7 (A5)
- net IR14: now also U16.6 (A6), U17.6 (A6), U24.6 (A6), U5.6 (A6)
- net IR15: now also U16.5 (A7), U17.5 (A7), U24.5 (A7), U5.5 (A7)
- net IR8: now also U16.12 (A0), U17.12 (A0), U24.12 (A0), U5.12 (A0)
- net IR9: now also U16.11 (A1), U17.11 (A1), U24.11 (A1), U5.11 (A1)
- net VCC: now also C11.1, C24.1, C25.1, C26.1, C27.1, C4.1, C5.1, C6.1, U16.31 (WE), U16.32 (VDD), U17.31 (WE), U17.32 (VDD), U24.31 (WE), U24.32 (VDD), U25.20 (VCC), U26.20 (VCC), U27.20 (VCC), U28.20 (VCC), U5.31 (WE), U5.32 (VDD)
- net ~A=B: now also U16.27 (A8), U17.27 (A8), U24.27 (A8), U5.27 (A8)
- net ~CarryOut: now also U16.26 (A9), U17.26 (A9), U24.26 (A9), U5.26 (A9)
- new net: U17.13 (DQ0), U27.2 (D0)
- new net: U17.14 (DQ1), U27.3 (D1)
- new net: U17.15 (DQ2), U27.4 (D2)
- new net: U17.17 (DQ3), U27.5 (D3)
- new net: U17.18 (DQ4), U27.6 (D4)
- new net: U17.19 (DQ5), U27.7 (D5)
- new net: U17.20 (DQ6), U27.8 (D6)
- new net: U17.21 (DQ7), U27.9 (D7)
- new net: U24.13 (DQ0), U28.2 (D0)
- new net: U24.14 (DQ1), U28.3 (D1)
- new net: U24.15 (DQ2), U28.4 (D2)
- new net: U24.17 (DQ3), U28.5 (D3)
- new net: U24.18 (DQ4), U28.6 (D4)
- new net: U24.19 (DQ5), U28.7 (D5)
- new net: U24.20 (DQ6), U28.8 (D6)
- new net: U24.21 (DQ7), U28.9 (D7)
- new net: U16.13 (DQ0), U26.2 (D0)
- new net: U16.14 (DQ1), U26.3 (D1)
- new net: U16.15 (DQ2), U26.4 (D2)
- new net: U16.17 (DQ3), U26.5 (D3)
- new net: U16.18 (DQ4), U26.6 (D4)
- new net: U16.19 (DQ5), U26.7 (D5)
- new net: U16.20 (DQ6), U26.8 (D6)
- new net: U16.21 (DQ7), U26.9 (D7)
- new net: U25.2 (D0), U5.13 (DQ0)
- new net: U25.3 (D1), U5.14 (DQ1)
- new net: U25.4 (D2), U5.15 (DQ2)
- new net: U25.5 (D3), U5.17 (DQ3)
- new net: U25.6 (D4), U5.18 (DQ4)
- new net: U25.7 (D5), U5.19 (DQ5)
- new net: U25.8 (D6), U5.20 (DQ6)
- new net: U25.9 (D7), U5.21 (DQ7)
- no-connect marks 11 -> 0
Other:
- note added: "ID/EX registers"
- note added: "Microcode ROM 1"
- note added: "Microcode ROM 2"
- note added: "Microcode ROM 3"
- note added: "Microcode ROM 4"
- moved on the sheet: C43, U47

Commit message: Merge branch "version2b".
This is a new version of the computer which incorporates a number of
improvements:
  * Uses a four layer PCB instead of six.
  * Replaced the clock with a new circuit. This is simpler, but allows for
    an external clock to be attached.
  * Changes to the ALU to have it operate over two clock cycles instead of
    one. This fixes a timing issue which makes the ALU unreliable at 10MHz.
  * Replaced instruction RAM with dual port SRAM.
  * Replaced the physical connector for expansion cards to interleave
    signals with ground.
  * Added places where components can be attached to provide AC termination
    of the data bus, should this be necessary.
Parts:
- U16: value GLS29EE010 -> Microcode ROM 3; footprint Package_DIP:DIP-32_W15.24mm_Socket -> Package_LCC:PLCC-32_THT-Socket
- U17: value GLS29EE010 -> Microcode ROM 2; footprint Package_DIP:DIP-32_W15.24mm_Socket -> Package_LCC:PLCC-32_THT-Socket
- U24: value GLS29EE010 -> Microcode ROM 1; footprint Package_DIP:DIP-32_W15.24mm_Socket -> Package_LCC:PLCC-32_THT-Socket
- U5: value GLS29EE010 -> Microcode ROM 4; footprint Package_DIP:DIP-32_W15.24mm_Socket -> Package_LCC:PLCC-32_THT-Socket
Connections:
- net ControlClock renamed ControlClock2
- net ControlClock2: no longer U47.11 (Cp)
- new net ControlClock0: U47.11 (Cp)
Other:
- note removed: "Microcode ROM 1"
- note removed: "Microcode ROM 2"
- note removed: "Microcode ROM 3"
- note removed: "Microcode ROM 4"
Changed lines of the file:
@@
 $Descr A2 23386 16535
 encoding utf-8
-Sheet 10 23
+Sheet 9 21
 Title "Instruction Decode"
 Date ""
@@
 IR7
 Text GLabel 16350 5250 0    50   Input ~ 0
-ControlClock
+ControlClock0
 $Comp
 L power:GND #PWR0129
@@
 AR Path="/5D2C0AA0/5DB5EC09" Ref="U?"  Part="1"
 AR Path="/5D2C0B92/5DB5EC09" Ref="U17"  Part="1"
-F 0 "U17" H 4050 7650 50  0000 C CNN
-F 1 "GLS29EE010" H 4050 7550 50  0000 C CNN
-F 2 "Package_DIP:DIP-32_W15.24mm_Socket" H 4400 7450 50  0001 C CNN
+F 0 "U17" H 3950 7650 50  0000 C CNN
+F 1 "Microcode ROM 2" H 3950 7550 50  0000 C CNN
+F 2 "Package_LCC:PLCC-32_THT-Socket" H 4400 7450 50  0001 C CNN
 F 3 "" H 4400 7450 50  0001 C CNN
 	1    4400 7450
@@
 AR Path="/5D2C0AA0/5DB5EC5B" Ref="U?"  Part="1"
 AR Path="/5D2C0B92/5DB5EC5B" Ref="U24"  Part="1"
-F 0 "U24" H 4050 10600 50  0000 C CNN
-F 1 "GLS29EE010" H 4050 10500 50  0000 C CNN
-F 2 "Package_DIP:DIP-32_W15.24mm_Socket" H 4400 10400 50  0001 C CNN
+F 0 "U24" H 3950 10600 50  0000 C CNN
+F 1 "Microcode ROM 1" H 3950 10500 50  0000 C CNN
+F 2 "Package_LCC:PLCC-32_THT-Socket" H 4400 10400 50  0001 C CNN
 F 3 "" H 4400 10400 50  0001 C CNN
 	1    4400 10400
@@
 IR[8..15]
 Text GLabel 2600 13600 0    50   Input ~ 0
-ControlClock
+ControlClock2
 $Comp
 L 74xx:74LS574 U?
@@
 Wire Bus Line
 	7150 7650 11200 7650
-Text Notes 2100 11250 0    50   ~ 0
-Microcode ROM 1
-Text Notes 2050 8300 0    50   ~ 0
-Microcode ROM 2
 $Comp
 L Memory_EEPROM:GLS29EE010 U?
@@
 AR Path="/5D2C0AA0/5EAAF06E" Ref="U?"  Part="1"
 AR Path="/5D2C0B92/5EAAF06E" Ref="U16"  Part="1"
-F 0 "U16" H 4050 4700 50  0000 C CNN
-F 1 "GLS29EE010" H 4050 4600 50  0000 C CNN
-F 2 "Package_DIP:DIP-32_W15.24mm_Socket" H 4400 4500 50  0001 C CNN
+F 0 "U16" H 3950 4700 50  0000 C CNN
+F 1 "Microcode ROM 3" H 3950 4600 50  0000 C CNN
+F 2 "Package_LCC:PLCC-32_THT-Socket" H 4400 4500 50  0001 C CNN
 F 3 "" H 4400 4500 50  0001 C CNN
 	1    4400 4500
@@
 Connection ~ 3050 8350
 Connection ~ 3150 8450
-Text Notes 2100 5650 0    50   ~ 0
-Microcode ROM 3
 $Comp
 L Memory_EEPROM:GLS29EE010 U?
@@
 AR Path="/5D2C0AA0/5EAAF07C" Ref="U?"  Part="1"
 AR Path="/5D2C0B92/5EAAF07C" Ref="U5"  Part="1"
-F 0 "U5" H 4050 1750 50  0000 C CNN
-F 1 "GLS29EE010" H 4050 1650 50  0000 C CNN
-F 2 "Package_DIP:DIP-32_W15.24mm_Socket" H 4400 1550 50  0001 C CNN
+F 0 "U5" H 3850 1750 50  0000 C CNN
+F 1 "Microcode ROM 4" H 3900 1650 50  0000 C CNN
+F 2 "Package_LCC:PLCC-32_THT-Socket" H 4400 1550 50  0001 C CNN
 F 3 "" H 4400 1550 50  0001 C CNN
 	1    4400 1550
@@
 Wire Wire Line
 	5100 2550 5400 2550
-Text Notes 2100 2700 0    50   ~ 0
-Microcode ROM 4
 Connection ~ 3050 5400
 Connection ~ 3150 5500
@@
 Wire Wire Line
 	9050 14600 8800 14600
-$Comp
-L power:VCC #PWR0212
-U 1 1 5DD15337
-P 3700 3450
-F 0 "#PWR0212" H 3700 3300 50  0001 C CNN
-F 1 "VCC" V 3718 3577 50  0000 L CNN
-F 2 "" H 3700 3450 50  0001 C CNN
-F 3 "" H 3700 3450 50  0001 C CNN
-	1    3700 3450
-	0    -1   -1   0
-$EndComp
 Connection ~ 11800 14300
 Connection ~ 11800 14600
@@
 Wire Bus Line
 	15200 9350 21100 9350
+$Comp
+L power:VCC #PWR0212
+U 1 1 5E058274
+P 3700 3450
+F 0 "#PWR0212" H 3700 3300 50  0001 C CNN
+F 1 "VCC" V 3718 3577 50  0000 L CNN
+F 2 "" H 3700 3450 50  0001 C CNN
+F 3 "" H 3700 3450 50  0001 C CNN
+	1    3700 3450
+	0    -1   -1   0
+$EndComp
 $EndSCHEMATC
