File: Schematics/Version2/SoundCard/VCA2.sch (KiCad schematic (older format))
At the start: 16 parts

Commit message: Sound card: Start assigning SMD footprints to schematic components.
Parts:
- U? (x2): footprint (none) -> Package_SO:SOIC-14_3.9x8.7mm_P1.27mm
- U? (x2): footprint Package_DIP:DIP-8_W7.62mm_Socket -> Package_SO:SOIC-8_3.9x4.9mm_P1.27mm
Changed lines of the file:
@@
 F 0 "U?" H 5300 4950 50  0000 C CNN
 F 1 "AS3360" H 5300 4850 50  0000 C CNN
-F 2 "" H 6300 3700 50  0001 C CNN
+F 2 "Package_SO:SOIC-14_3.9x8.7mm_P1.27mm" H 6300 3700 50  0001 C CNN
 F 3 "http://www.alfarzpp.lv/eng/sc/AS3360.pdf" H 6250 3750 50  0001 C CNN
 	2    5600 4400
@@
 F 0 "U?" H 5250 3200 50  0000 C CNN
 F 1 "AS3360" H 5250 3100 50  0000 C CNN
-F 2 "" H 6300 1900 50  0001 C CNN
+F 2 "Package_SO:SOIC-14_3.9x8.7mm_P1.27mm" H 6300 1900 50  0001 C CNN
 F 3 "http://www.alfarzpp.lv/eng/sc/AS3360.pdf" H 6250 1950 50  0001 C CNN
 	1    5600 2600
@@
 F 0 "U?" H 7950 3150 50  0000 C CNN
 F 1 "TL072" H 7950 3050 50  0000 C CNN
-F 2 "Package_DIP:DIP-8_W7.62mm_Socket" H 7950 2800 50  0001 C CNN
+F 2 "Package_SO:SOIC-8_3.9x4.9mm_P1.27mm" H 7950 2800 50  0001 C CNN
 F 3 "http://www.ti.com/lit/ds/symlink/tl071.pdf" H 7950 2800 50  0001 C CNN
 	1    7950 2800
@@
 F 0 "U?" H 8200 4750 50  0000 C CNN
 F 1 "TL072" H 8200 4850 50  0000 C CNN
-F 2 "Package_DIP:DIP-8_W7.62mm_Socket" H 8200 5100 50  0001 C CNN
+F 2 "Package_SO:SOIC-8_3.9x4.9mm_P1.27mm" H 8200 5100 50  0001 C CNN
 F 3 "http://www.ti.com/lit/ds/symlink/tl071.pdf" H 8200 5100 50  0001 C CNN
 	2    8200 5100

Commit message: Sound card: add the Electric Druid Noise 1B digital sound generator.
The gain on the noise voice is controlled by one of the AS3360 units.
The master gain control is removed in order to make this possible.
Parts:
- U12: renamed from U?; footprint Package_DIP:DIP-8_W7.62mm_Socket -> Package_SO:SOIC-8_3.9x4.9mm_P1.27mm
- gave numbers to parts that had none: 13

Commit message: Sound Card: Finish routing SMD PCB for rev 2
Parts:
- C9: footprint (none) -> Capacitor_SMD:C_0603_1608Metric_Pad1.05x0.95mm_HandSolder
- R48, R49, R50, R51, R52, R53: footprint (none) -> Resistor_SMD:R_0603_1608Metric_Pad1.05x0.95mm_HandSolder
- R54, R55, R56, R57: footprint Resistor_THT:R_Axial_DIN0207_L6.3mm_D2.5mm_P7.62mm_Horizontal -> Resistor_SMD:R_0603_1608Metric_Pad1.05x0.95mm_HandSolder
Changed lines of the file:
@@
 F 0 "R53" H 6318 4696 50  0000 L CNN
 F 1 "47kΩ" H 6318 4605 50  0000 L CNN
-F 2 "" V 6290 4640 50  0001 C CNN
+F 2 "Resistor_SMD:R_0603_1608Metric_Pad1.05x0.95mm_HandSolder" V 6290 4640 50  0001 C CNN
 F 3 "~" H 6250 4650 50  0001 C CNN
 	1    6250 4650
@@
 F 0 "R51" H 4168 3746 50  0000 L CNN
 F 1 "2.4kΩ" H 4168 3655 50  0000 L CNN
-F 2 "" V 4140 3690 50  0001 C CNN
+F 2 "Resistor_SMD:R_0603_1608Metric_Pad1.05x0.95mm_HandSolder" V 4140 3690 50  0001 C CNN
 F 3 "~" H 4100 3700 50  0001 C CNN
 	1    4100 3700
@@
 F 0 "R49" V 3395 4200 50  0000 C CNN
 F 1 "16kΩ" V 3486 4200 50  0000 C CNN
-F 2 "" V 3640 4190 50  0001 C CNN
+F 2 "Resistor_SMD:R_0603_1608Metric_Pad1.05x0.95mm_HandSolder" V 3640 4190 50  0001 C CNN
 F 3 "~" H 3600 4200 50  0001 C CNN
 	1    3600 4200
@@
 F 0 "C9" H 5065 3096 50  0000 L CNN
 F 1 "5nF" H 5065 3005 50  0000 L CNN
-F 2 "" H 4988 2900 50  0001 C CNN
+F 2 "Capacitor_SMD:C_0603_1608Metric_Pad1.05x0.95mm_HandSolder" H 4988 2900 50  0001 C CNN
 F 3 "~" H 4950 3050 50  0001 C CNN
 	1    4950 3050
@@
 F 0 "R48" V 3395 2400 50  0000 C CNN
 F 1 "16kΩ" V 3486 2400 50  0000 C CNN
-F 2 "" V 3640 2390 50  0001 C CNN
+F 2 "Resistor_SMD:R_0603_1608Metric_Pad1.05x0.95mm_HandSolder" V 3640 2390 50  0001 C CNN
 F 3 "~" H 3600 2400 50  0001 C CNN
 	1    3600 2400
@@
 F 0 "R50" H 4032 2854 50  0000 R CNN
 F 1 "2.4kΩ" H 4032 2945 50  0000 R CNN
-F 2 "" V 4140 2890 50  0001 C CNN
+F 2 "Resistor_SMD:R_0603_1608Metric_Pad1.05x0.95mm_HandSolder" V 4140 2890 50  0001 C CNN
 F 3 "~" H 4100 2900 50  0001 C CNN
 	1    4100 2900
@@
 F 0 "R52" H 6318 2896 50  0000 L CNN
 F 1 "47kΩ" H 6318 2805 50  0000 L CNN
-F 2 "" V 6290 2840 50  0001 C CNN
+F 2 "Resistor_SMD:R_0603_1608Metric_Pad1.05x0.95mm_HandSolder" V 6290 2840 50  0001 C CNN
 F 3 "~" H 6250 2850 50  0001 C CNN
 	1    6250 2850
@@
 F 0 "R54" V 7355 3350 50  0000 C CNN
 F 1 "10kΩ" V 7264 3350 50  0000 C CNN
-F 2 "Resistor_THT:R_Axial_DIN0207_L6.3mm_D2.5mm_P7.62mm_Horizontal" V 7190 3340 50  0001 C CNN
+F 2 "Resistor_SMD:R_0603_1608Metric_Pad1.05x0.95mm_HandSolder" V 7190 3340 50  0001 C CNN
 F 3 "~" H 7150 3350 50  0001 C CNN
 	1    7150 3350
@@
 F 0 "R56" V 8155 3350 50  0000 C CNN
 F 1 "20kΩ" V 8064 3350 50  0000 C CNN
-F 2 "Resistor_THT:R_Axial_DIN0207_L6.3mm_D2.5mm_P7.62mm_Horizontal" V 7990 3340 50  0001 C CNN
+F 2 "Resistor_SMD:R_0603_1608Metric_Pad1.05x0.95mm_HandSolder" V 7990 3340 50  0001 C CNN
 F 3 "~" H 7950 3350 50  0001 C CNN
 	1    7950 3350
@@
 F 0 "R55" V 7555 4500 50  0000 C CNN
 F 1 "10kΩ" V 7464 4500 50  0000 C CNN
-F 2 "Resistor_THT:R_Axial_DIN0207_L6.3mm_D2.5mm_P7.62mm_Horizontal" V 7390 4490 50  0001 C CNN
+F 2 "Resistor_SMD:R_0603_1608Metric_Pad1.05x0.95mm_HandSolder" V 7390 4490 50  0001 C CNN
 F 3 "~" H 7350 4500 50  0001 C CNN
 	1    7350 4500
@@
 F 0 "R57" V 8355 4500 50  0000 C CNN
 F 1 "4.7kΩ" V 8264 4500 50  0000 C CNN
-F 2 "Resistor_THT:R_Axial_DIN0207_L6.3mm_D2.5mm_P7.62mm_Horizontal" V 8190 4490 50  0001 C CNN
+F 2 "Resistor_SMD:R_0603_1608Metric_Pad1.05x0.95mm_HandSolder" V 8190 4490 50  0001 C CNN
 F 3 "~" H 8150 4500 50  0001 C CNN
 	1    8150 4500
